File: kicad/battlepoint.kicad_pcb (KiCad board)
At the start: 2 copper layers, 101.6 x 154.9 mm, 20 parts, among them J1 BTNS, J2 TMR_LEDS, J3 CAP_LEDS, P12 PANEL_OUT, P13 PANEL_IN, P14 OLED_OUT, P5 SPK, P8 AUDIO_JACK, SW1 BTN_UP, SW2 BTN_DWN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

Commit message: made button board fit
Parts:
- removed P12: PANEL_OUT, Connectors_JST:JST_XH_B05B-XH-A_05x2.50mm_Straight
- added P17: BTNS_OUT, Pin_Headers:Pin_Header_Straight_1x04, F.Cu at (76.8, 170.8)
- P13: value PANEL_IN -> BTNS_IN; footprint Connectors_JST:JST_XH_B05B-XH-A_05x2.50mm_Straight -> Pin_Headers:Pin_Header_Straight_1x04
- moved R6 92.0 mm to (81.9, 178.4)
- moved R7 91.6 mm to (76.8, 175.3), turned to 0 degrees
- moved P14 78.1 mm to (66.0, 172.7)
- moved R5 72.5 mm to (82.5, 161.9), turned to 270 degrees
- moved R3 65.0 mm to (90.8, 158.1), turned to 90 degrees
- moved R4 63.8 mm to (85.1, 155.6)
- moved SW2 57.4 mm to (95.2, 99.7), turned to 90 degrees
- moved SW3 57.4 mm to (104.1, 99.7), turned to 90 degrees
- moved SW1 57.4 mm to (86.4, 99.7), turned to 90 degrees
- moved P13 55.8 mm to (108.6, 92.7), turned to 0 degrees
Connections:
- P13 pad 1: +5V -> GND
- P14 pad 2: Net-(P13-Pad3) -> SCL
- P14 pad 3: Net-(P13-Pad4) -> SDA
- R3 pad 2: Net-(P13-Pad2) -> A0
- R4 pad 1: Net-(P13-Pad2) -> A0
- R4 pad 2: Net-(R4-Pad2) -> Net-(P17-Pad4)
- R5 pad 1: Net-(R4-Pad2) -> Net-(P17-Pad4)
- R5 pad 2: Net-(R5-Pad2) -> Net-(P17-Pad3)
- R6 pad 1: Net-(R5-Pad2) -> Net-(P17-Pad3)
- R7 pad 2: Net-(R7-Pad2) -> Net-(P17-Pad2)
- SW1 pad 1: Net-(R4-Pad2) -> Net-(P13-Pad4)
- SW2 pad 1: Net-(R5-Pad2) -> Net-(P13-Pad3)
- SW3 pad 1: Net-(R7-Pad2) -> Net-(P13-Pad2)
Routing:
- net Net-(R4-Pad2): track 51.8 -> 0.00 mm
- net A0: track 44.6 -> 16.6 mm
- net Net-(R5-Pad2): track 27.9 -> 0.00 mm
- net +5V: track 187.7 -> 169.8 mm
- net Net-(P17-Pad4): track 0.00 -> 16.6 mm
- net Net-(P13-Pad4): track 16.7 -> 32.6 mm
- net Net-(P17-Pad3): track 0.00 -> 15.3 mm
- net Net-(R7-Pad2): track 11.8 -> 0.00 mm
- net SDA: track 27.5 -> 18.1 mm
- net SCL: track 30.1 -> 21.2 mm
- net Net-(P13-Pad3): track 19.1 -> 24.7 mm
- net Net-(P13-Pad2): track 17.8 -> 12.4 mm
- net Net-(P17-Pad2): track 0.00 -> 4.46 mm
- net GND: track 303.9 -> 305.4 mm
Other:
- outline, holes or cut-outs redrawn
