File: kicad/battlepoint.sch (KiCad schematic (older format))
At the start: 13 parts, among them J1 Arduino1, J2 Arduino2, J3 Arduino3, J4 Arduino4, J5 PANEL, J6 SWITCHES, J7 Barrel_Jack, J8 LIGHTS, U1 LM7805_TO220

Commit message: working mostly
Parts:
- removed C1: 0.1uf, Capacitors_THT:C_Rect_L7.0mm_W2.5mm_P5.00mm, symbol C
- removed C2: 22uf, Capacitors_THT:CP_Radial_D4.0mm_P1.50mm, symbol CP
- removed J1: Arduino1, Socket_Strips:Socket_Strip_Straight_1x06_Pitch2.54mm, symbol Conn_01x06_Female
- removed J2: Arduino2, Socket_Strips:Socket_Strip_Straight_1x06_Pitch2.54mm, symbol Conn_01x06_Female
- removed J3: Arduino3, Socket_Strips:Socket_Strip_Straight_1x08_Pitch2.54mm, symbol Conn_01x08_Female
- removed J4: Arduino4, Socket_Strips:Socket_Strip_Straight_1x08_Pitch2.54mm, symbol Conn_01x08_Female
- removed J5: PANEL, Connectors:RJ45_8, symbol RJ45
- removed J6: SWITCHES, Connectors:RJ45_8, symbol RJ45
- removed J7: Barrel_Jack, Connectors:BARREL_JACK, symbol Barrel_Jack
- removed J8: LIGHTS, Connectors:RJ45_8, symbol RJ45
- removed U1: LM7805_TO220, TO_SOT_Packages_THT:TO-220-3_Vertical, symbol LM7805_TO220
- added ARD1: UNO_SHIELD, Arduino:Arduino_Uno_Shield, symbol Arduino_Uno_Shield
- added J1: BTNS, Connect:RJ45_8, symbol RJ45
- added P1: TMR1_LED, Connect:USB_A, symbol USB_A
- added P10: OLED, Connectors_JST:JST_XH_B04B-XH-A_04x2.50mm_Straight, symbol CONN_01X04
- added P2: TMR2_LED, Connect:USB_A, symbol USB_A
- added P3: CAP_LED, Connect:USB_A, symbol USB_A
- added P4: OWN_LED, Connect:USB_A, symbol USB_A
- added P5: SPK, Connectors_JST:JST_XH_B02B-XH-A_02x2.50mm_Straight, symbol CONN_01X02
- added P8: AUDIO_JACK, Connectors_JST:JST_XH_B04B-XH-A_04x2.50mm_Straight, symbol CONN_01X04
- added P9: KEYPAD, Connectors_JST:JST_XH_B03B-XH-A_03x2.50mm_Straight, symbol CONN_01X03
- added R3: 2K, symbol R
- added R4: 330, symbol R
- added R5: 620, symbol R
- added R6: 1K, symbol R
- added R7: 3.3K, symbol R
- added SW1: BTN_UP, Buttons_Switches_ThroughHole:SW_PUSH_6mm, symbol SW_PUSH
- added SW2: BTN_DWN, Buttons_Switches_ThroughHole:SW_PUSH_6mm, symbol SW_PUSH
- added SW3: BTN_SEL, Buttons_Switches_ThroughHole:SW_PUSH_6mm, symbol SW_PUSH
- added U1: DFPLAYER_MINI, Arduino:dfplayer_mini, symbol DFPLAYER_MINI
- R1, R2: footprint Resistors_THT:R_Axial_DIN0204_L3.6mm_D1.6mm_P2.54mm_Vertical -> Resistors_ThroughHole:Resistor_Horizontal_RM7mm
Connections:
- net labels added: D10, D11, D12, D13, D2, D3, D4, D5, D6, D7, D8, D9, KEYPAD, SCL, SDA
- net labels removed: +VDC, 3.3V, 5V, A1, A2, A3, A5, P0, P1, P10, P11, P12, P13, P14, P15, P2, P3, P4, P5, P6, P7, P8, P9, RESET, VIN
- wire segments 82 -> 95
- no-connect marks 3 -> 10

Commit message: progress
Parts:
- removed P10: OLED, Connectors_JST:JST_XH_B04B-XH-A_04x2.50mm_Straight, symbol CONN_01X04
- removed P9: KEYPAD, Connectors_JST:JST_XH_B03B-XH-A_03x2.50mm_Straight, symbol CONN_01X03
- added P12: PANEL_OUT, Connectors_JST:JST_XH_B05B-XH-A_05x2.50mm_Straight, symbol CONN_01X05
- added P13: PANEL_IN, Connectors_JST:JST_XH_B05B-XH-A_05x2.50mm_Straight, symbol CONN_01X05
- added P14: OLED_OUT, Connectors_JST:JST_XH_B04B-XH-A_04x2.50mm_Straight, symbol CONN_01X04
- R3, R4, R5, R6, R7: footprint (none) -> Resistors_ThroughHole:Resistor_Horizontal_RM7mm
Connections:
- net labels removed: KEYPAD
- wire segments 95 -> 101

Commit message: about to start routing
Connections:
- net SCL: now also ARD1.SCL
- net SDA: now also ARD1.SDA

Commit message: finished for now i think
Parts:
- R3, R4, R5, R6, R7: footprint Resistors_ThroughHole:Resistor_Horizontal_RM7mm -> Resistors_ThroughHole:Resistor_Vertical_RM5mm
Connections:
- net A4: now also ARD1.A4
- net at P8.4 (P4), U1.6 (SPK_1): now also P8.2 (P2)
- no-connect marks 10 -> 11
Changed lines of the file:
@@
 F 0 "R3" V 9180 3200 50  0000 C CNN
 F 1 "2K" V 9100 3200 50  0000 C CNN
-F 2 "Resistors_ThroughHole:Resistor_Horizontal_RM7mm" V 9030 3200 50  0001 C CNN
+F 2 "Resistors_ThroughHole:Resistor_Vertical_RM5mm" V 9030 3200 50  0001 C CNN
 F 3 "" H 9100 3200 50  0000 C CNN
 	1    9100 3200
@@
 F 0 "R4" V 9180 3700 50  0000 C CNN
 F 1 "330" V 9100 3700 50  0000 C CNN
-F 2 "Resistors_ThroughHole:Resistor_Horizontal_RM7mm" V 9030 3700 50  0001 C CNN
+F 2 "Resistors_ThroughHole:Resistor_Vertical_RM5mm" V 9030 3700 50  0001 C CNN
 F 3 "" H 9100 3700 50  0000 C CNN
 	1    9100 3700
@@
 F 0 "R5" V 9180 4200 50  0000 C CNN
 F 1 "620" V 9100 4200 50  0000 C CNN
-F 2 "Resistors_ThroughHole:Resistor_Horizontal_RM7mm" V 9030 4200 50  0001 C CNN
+F 2 "Resistors_ThroughHole:Resistor_Vertical_RM5mm" V 9030 4200 50  0001 C CNN
 F 3 "" H 9100 4200 50  0000 C CNN
 	1    9100 4200
@@
 F 0 "R6" V 9180 4650 50  0000 C CNN
 F 1 "1K" V 9100 4650 50  0000 C CNN
-F 2 "Resistors_ThroughHole:Resistor_Horizontal_RM7mm" V 9030 4650 50  0001 C CNN
+F 2 "Resistors_ThroughHole:Resistor_Vertical_RM5mm" V 9030 4650 50  0001 C CNN
 F 3 "" H 9100 4650 50  0000 C CNN
 	1    9100 4650
@@
 F 0 "R7" V 9180 5050 50  0000 C CNN
 F 1 "3.3K" V 9100 5050 50  0000 C CNN
-F 2 "Resistors_ThroughHole:Resistor_Horizontal_RM7mm" V 9030 5050 50  0001 C CNN
+F 2 "Resistors_ThroughHole:Resistor_Vertical_RM5mm" V 9030 5050 50  0001 C CNN
 F 3 "" H 9100 5050 50  0000 C CNN
 	1    9100 5050
@@
 	5400 2000 5400 2100
 Wire Wire Line
-	5500 2000 5500 2050
-Wire Wire Line
-	5500 2050 6250 2050
-Wire Wire Line
-	6250 2050 6250 2000
-Wire Wire Line
-	6350 2000 6350 2050
-Wire Wire Line
-	6350 2050 7350 2050
-Wire Wire Line
-	7450 2050 7450 2100
-Wire Wire Line
-	7450 2100 8200 2100
-Wire Wire Line
-	8200 2100 8200 2050
+	8200 2050 8200 2700
 Wire Wire Line
 	2850 1900 3050 1900
@@
 Wire Wire Line
 	2000 2150 2050 2150
-Wire Wire Line
-	2350 2300 3050 2300
-Wire Wire Line
-	2600 2300 2600 2500
-Wire Wire Line
-	2600 2500 2150 2500
-Wire Wire Line
-	2150 2500 2150 2150
-Wire Wire Line
-	2350 2300 2350 2150
-Wire Wire Line
-	2000 2500 2100 2500
-Wire Wire Line
-	2100 2500 2100 2600
-Wire Wire Line
-	2100 2600 2250 2600
-Wire Wire Line
-	2250 2600 2250 2150
 Wire Wire Line
 	800  1550 800  1950
@@
 Wire Wire Line
 	1600 3700 1900 3700
+NoConn ~ 8300 2050
+Wire Wire Line
+	5500 2000 5500 2700
+Wire Wire Line
+	5500 2700 6250 2700
+Wire Wire Line
+	6250 2700 6250 2000
+Wire Wire Line
+	6350 2000 6350 2700
+Wire Wire Line
+	6350 2700 7350 2700
+Wire Wire Line
+	7350 2700 7350 2050
+Wire Wire Line
+	7450 2050 7450 2700
+Wire Wire Line
+	7450 2700 8200 2700
+Wire Wire Line
+	3050 2300 2150 2300
+Wire Wire Line
+	2150 2300 2150 2150
+Connection ~ 2350 2300
+Wire Wire Line
+	2350 2150 2350 2300
+Connection ~ 2250 2700
+Wire Wire Line
+	2250 2150 2250 2700
+Text GLabel 1600 4100 0    60   Input ~ 0
+A4
+Wire Wire Line
+	1600 4100 1900 4100
 $EndSCHEMATC

Commit message: used rj45s for connections
Parts:
- removed P1: TMR1_LED, Connect:USB_A, symbol USB_A
- removed P2: TMR2_LED, Connect:USB_A, symbol USB_A
- removed P3: CAP_LED, Connect:USB_A, symbol USB_A
- removed P4: OWN_LED, Connect:USB_A, symbol USB_A
- added J2: TMR_LEDS, Connect:RJ45_8, symbol RJ45
- added J3: CAP_LEDS, Connect:RJ45_8, symbol RJ45
Connections:
- net +5V: now also J2.1, J2.8, J3.1, J3.8
- net D10: now also J1.4; no longer J1.8
- net D11: now also J1.8; no longer J1.4
- net D5: now also J2.2
- net GND: now also J2.4, J2.5, J3.4, J3.5
- new net: J2.3, J2.7
- new net: J2.6, J3.2
- new net: J3.3, J3.7
Changed lines of the file:
@@
-$EndComp
-$Comp
-L USB_A P1
-U 1 1 5A288AA4
-P 6350 1700
-F 0 "P1" H 6550 1500 50  0000 C CNN
-F 1 "TMR1_LED" H 6300 1900 50  0000 C CNN
-F 2 "Connect:USB_A" V 6300 1600 50  0001 C CNN
-F 3 "" V 6300 1600 50  0000 C CNN
-	1    6350 1700
-	1    0    0    -1
-$EndComp
-$Comp
-L USB_A P2
-U 1 1 5A288B61
-P 7450 1750
-F 0 "P2" H 7650 1550 50  0000 C CNN
-F 1 "TMR2_LED" H 7400 1950 50  0000 C CNN
-F 2 "Connect:USB_A" V 7400 1650 50  0001 C CNN
-F 3 "" V 7400 1650 50  0000 C CNN
-	1    7450 1750
-	1    0    0    -1
-$EndComp
-$Comp
-L USB_A P3
-U 1 1 5A288BC4
-P 5500 1700
-F 0 "P3" H 5700 1500 50  0000 C CNN
-F 1 "CAP_LED" H 5450 1900 50  0000 C CNN
-F 2 "Connect:USB_A" V 5450 1600 50  0001 C CNN
-F 3 "" V 5450 1600 50  0000 C CNN
-	1    5500 1700
-	1    0    0    -1
-$EndComp
-$Comp
-L USB_A P4
-U 1 1 5A288C1F
-P 8300 1750
-F 0 "P4" H 8500 1550 50  0000 C CNN
-F 1 "OWN_LED" H 8250 1950 50  0000 C CNN
-F 2 "Connect:USB_A" V 8250 1650 50  0001 C CNN
-F 3 "" V 8250 1650 50  0000 C CNN
-	1    8300 1750
-	1    0    0    -1
 $EndComp
 $Comp
@@
 L GND #PWR02
 U 1 1 5A28A37E
-P 5600 2250
-F 0 "#PWR02" H 5600 2000 50  0001 C CNN
-F 1 "GND" H 5600 2100 50  0000 C CNN
-F 2 "" H 5600 2250 50  0000 C CNN
-F 3 "" H 5600 2250 50  0000 C CNN
-	1    5600 2250
+P 5550 2100
+F 0 "#PWR02" H 5550 1850 50  0001 C CNN
+F 1 "GND" H 5550 1950 50  0000 C CNN
+F 2 "" H 5550 2100 50  0000 C CNN
+F 3 "" H 5550 2100 50  0000 C CNN
+	1    5550 2100
 	1    0    0    -1
 $EndComp
@@
 L GND #PWR03
 U 1 1 5A28A3B3
-P 6450 2250
-F 0 "#PWR03" H 6450 2000 50  0001 C CNN
-F 1 "GND" H 6450 2100 50  0000 C CNN
-F 2 "" H 6450 2250 50  0000 C CNN
-F 3 "" H 6450 2250 50  0000 C CNN
-	1    6450 2250
+P 5650 2100
+F 0 "#PWR03" H 5650 1850 50  0001 C CNN
+F 1 "GND" H 5650 1950 50  0000 C CNN
+F 2 "" H 5650 2100 50  0000 C CNN
+F 3 "" H 5650 2100 50  0000 C CNN
+	1    5650 2100
 	1    0    0    -1
 $EndComp
@@
 L +5V #PWR010
 U 1 1 5A28A59C
-P 5300 2200
-F 0 "#PWR010" H 5300 2050 50  0001 C CNN
-F 1 "+5V" H 5300 2340 50  0000 C CNN
-F 2 "" H 5300 2200 50  0000 C CNN
-F 3 "" H 5300 2200 50  0000 C CNN
-	1    5300 2200
+P 5250 2250
+F 0 "#PWR010" H 5250 2100 50  0001 C CNN
+F 1 "+5V" H 5250 2390 50  0000 C CNN
+F 2 "" H 5250 2250 50  0000 C CNN
+F 3 "" H 5250 2250 50  0000 C CNN
+	1    5250 2250
 	-1   0    0    1
 $EndComp
@@
 L GND #PWR011
 U 1 1 5A28ACCE
-P 7550 2250
-F 0 "#PWR011" H 7550 2000 50  0001 C CNN
-F 1 "GND" H 7550 2100 50  0000 C CNN
-F 2 "" H 7550 2250 50  0000 C CNN
-F 3 "" H 7550 2250 50  0000 C CNN
-	1    7550 2250
+P 7300 2100
+F 0 "#PWR011" H 7300 1850 50  0001 C CNN
+F 1 "GND" H 7300 1950 50  0000 C CNN
+F 2 "" H 7300 2100 50  0000 C CNN
+F 3 "" H 7300 2100 50  0000 C CNN
+	1    7300 2100
 	1    0    0    -1
 $EndComp
@@
 L GND #PWR012
 U 1 1 5A28AD03
-P 8400 2250
-F 0 "#PWR012" H 8400 2000 50  0001 C CNN
-F 1 "GND" H 8400 2100 50  0000 C CNN
-F 2 "" H 8400 2250 50  0000 C CNN
-F 3 "" H 8400 2250 50  0000 C CNN
-	1    8400 2250
+P 7400 2100
+F 0 "#PWR012" H 7400 1850 50  0001 C CNN
+F 1 "GND" H 7400 1950 50  0000 C CNN
+F 2 "" H 7400 2100 50  0000 C CNN
+F 3 "" H 7400 2100 50  0000 C CNN
+	1    7400 2100
 	1    0    0    -1
 $EndComp
@@
 L +5V #PWR013
 U 1 1 5A28AE34
-P 6150 2250
-F 0 "#PWR013" H 6150 2100 50  0001 C CNN
-F 1 "+5V" H 6150 2390 50  0000 C CNN
-F 2 "" H 6150 2250 50  0000 C CNN
-F 3 "" H 6150 2250 50  0000 C CNN
-	1    6150 2250
+P 5950 2200
+F 0 "#PWR013" H 5950 2050 50  0001 C CNN
+F 1 "+5V" H 5950 2340 50  0000 C CNN
+F 2 "" H 5950 2200 50  0000 C CNN
+F 3 "" H 5950 2200 50  0000 C CNN
+	1    5950 2200
 	-1   0    0    1
 $EndComp
@@
 L +5V #PWR014
 U 1 1 5A28AE69
-P 7250 2250
-F 0 "#PWR014" H 7250 2100 50  0001 C CNN
-F 1 "+5V" H 7250 2390 50  0000 C CNN
-F 2 "" H 7250 2250 50  0000 C CNN
-F 3 "" H 7250 2250 50  0000 C CNN
-	1    7250 2250
+P 7000 2100
+F 0 "#PWR014" H 7000 1950 50  0001 C CNN
+F 1 "+5V" H 7000 2240 50  0000 C CNN
+F 2 "" H 7000 2100 50  0000 C CNN
+F 3 "" H 7000 2100 50  0000 C CNN
+	1    7000 2100
 	-1   0    0    1
 $EndComp
@@
 L +5V #PWR015
 U 1 1 5A28AE9E
-P 8100 2250
-F 0 "#PWR015" H 8100 2100 50  0001 C CNN
-F 1 "+5V" H 8100 2390 50  0000 C CNN
-F 2 "" H 8100 2250 50  0000 C CNN
-F 3 "" H 8100 2250 50  0000 C CNN
-	1    8100 2250
+P 7700 2100
+F 0 "#PWR015" H 7700 1950 50  0001 C CNN
+F 1 "+5V" H 7700 2240 50  0000 C CNN
+F 2 "" H 7700 2100 50  0000 C CNN
+F 3 "" H 7700 2100 50  0000 C CNN
+	1    7700 2100
 	-1   0    0    1
 $EndComp
@@
 Text GLabel 5800 4700 0    60   Input ~ 0
 A0
-Text GLabel 5400 2100 3    60   Input ~ 0
+Text GLabel 5350 2050 3    60   Input ~ 0
 D5
-Text GLabel 1500 1650 3    60   Input ~ 0
+Text GLabel 1100 1650 3    60   Input ~ 0
 D10
-Text GLabel 1100 1650 3    60   Input ~ 0
+Text GLabel 1500 1700 3    60   Input ~ 0
 D11
 Text GLabel 2850 1900 0    60   Input ~ 0
@@
 	4500 4400 4750 4400
 Wire Wire Line
-	5600 2000 5600 2250
-Wire Wire Line
-	6450 2000 6450 2250
-Wire Wire Line
-	7550 2050 7550 2250
-Wire Wire Line
-	8400 2050 8400 2250
-Wire Wire Line
-	6150 2000 6150 2250
-Wire Wire Line
-	5300 2000 5300 2200
-Wire Wire Line
-	7250 2050 7250 2250
-Wire Wire Line
-	8100 2050 8100 2250
-Wire Wire Line
-	5400 2000 5400 2100
-Wire Wire Line
-	8200 2050 8200 2700
-Wire Wire Line
 	2850 1900 3050 1900
 Wire Wire Line
@@
 	1000 1550 1000 1650
 Wire Wire Line
-	1100 1550 1100 1650
-Wire Wire Line
 	1200 1550 1200 1950
 Wire Wire Line
@@
 Wire Wire Line
 	1400 1550 1400 1650
-Wire Wire Line
-	1500 1550 1500 1650
 Wire Wire Line
 	3150 6250 3150 6400
@@
 Wire Wire Line
 	1600 3700 1900 3700
-NoConn ~ 8300 2050
-Wire Wire Line
-	5500 2000 5500 2700
-Wire Wire Line
-	5500 2700 6250 2700
-Wire Wire Line
-	6250 2700 6250 2000
-Wire Wire Line
-	6350 2000 6350 2700
-Wire Wire Line
-	6350 2700 7350 2700
-Wire Wire Line
-	7350 2700 7350 2050
-Wire Wire Line
-	7450 2050 7450 2700
-Wire Wire Line
-	7450 2700 8200 2700
 Wire Wire Line
 	3050 2300 2150 2300
@@
 Wire Wire Line
 	1600 4100 1900 4100
+$Comp
+L RJ45 J2
+U 1 1 5A2B570A
+P 5600 1450
+F 0 "J2" H 5800 1950 50  0000 C CNN
+F 1 "TMR_LEDS" H 5450 1950 50  0000 C CNN
+F 2 "Connect:RJ45_8" H 5600 1450 50  0001 C CNN
+F 3 "" H 5600 1450 50  0000 C CNN
+	1    5600 1450
+	1    0    0    -1
+$EndComp
+$Comp
+L RJ45 J3
+U 1 1 5A2B57CE
+P 7350 1450
+F 0 "J3" H 7550 1950 50  0000 C CNN
+F 1 "CAP_LEDS" H 7200 1950 50  0000 C CNN
+F 2 "Connect:RJ45_8" H 7350 1450 50  0001 C CNN
+F 3 "" H 7350 1450 50  0000 C CNN
+	1    7350 1450
+	1    0    0    -1
+$EndComp
+Wire Wire Line
+	5250 1900 5250 2250
+Wire Wire Line
+	5350 1900 5350 2050
+Wire Wire Line
+	5550 1900 5550 2100
+Wire Wire Line
+	7000 1900 7000 2100
+Wire Wire Line
+	1100 1650 1100 1550
+Wire Wire Line
+	1500 1700 1500 1550
+Wire Wire Line
+	7700 1900 7700 2100
+Wire Wire Line
+	7400 1900 7400 2100
+Wire Wire Line
+	7300 1900 7300 2100
+Wire Wire Line
+	5650 1900 5650 2100
+Wire Wire Line
+	5950 1900 5950 2200
+Wire Wire Line
+	5450 1900 5450 2550
+Wire Wire Line
+	5450 2550 5850 2550
+Wire Wire Line
+	5850 2550 5850 1900
+Wire Wire Line
+	5750 1900 5750 2050
+Wire Wire Line
+	5750 2050 7100 2050
+Wire Wire Line
+	7100 2050 7100 1900
+NoConn ~ 7500 1900
+Wire Wire Line
+	7200 1900 7200 2500
+Wire Wire Line
+	7200 2500 7600 2500
+Wire Wire Line
+	7600 2500 7600 1900
 $EndSCHEMATC

Commit message: made button board fit
Parts:
- removed P12: PANEL_OUT, Connectors_JST:JST_XH_B05B-XH-A_05x2.50mm_Straight, symbol CONN_01X05
- removed P13: PANEL_IN, Connectors_JST:JST_XH_B05B-XH-A_05x2.50mm_Straight, symbol CONN_01X05
- added P13: BTNS_IN, Pin_Headers:Pin_Header_Straight_1x04, symbol CONN_01X04
- added P17: BTNS_OUT, Pin_Headers:Pin_Header_Straight_1x04, symbol CONN_01X04
Connections:
- net A0: now also R3.2, R4.1
- net GND: now also P13.1 (P1), P17.1 (P1)
- net SCL: now also P14.2 (P2)
- net SDA: now also P14.3 (P3)
- net at R4.2, R5.1: now also P17.4 (P4); no longer SW1.1
- net at R5.2, R6.1: now also P17.3 (P3); no longer SW2.1
- net at SW3.1: now also P13.2 (P2); no longer R7.2
- new net: P13.4 (P4), SW1.1
- new net: P13.3 (P3), SW2.1
- new net: P17.2 (P2), R7.2
Other:
- moved on the sheet: P14, R3, R4, R5, R6, R7

Commit message: base version without regulator
Parts:
- added R10: 1K, Resistors_ThroughHole:Resistor_Horizontal_RM7mm, symbol R
Connections:
- net A4: no longer ARD1.A4, R1.2, R2.1
- net D8: now also R10.2; no longer U1.2 (RX)
- net A2: now reaches ARD1.A2
- net A2: now also R1.2, R2.1
- new net: R10.1, U1.2 (RX)
Changed lines of the file:
@@
 LIBS:arduino
 LIBS:rur
+LIBS:battlepoint-cache
 EELAYER 25 0
 EELAYER END
@@
 Text GLabel 1500 1700 3    60   Input ~ 0
 D11
-Text GLabel 2850 1900 0    60   Input ~ 0
+Text GLabel 2650 1900 0    60   Input ~ 0
 D8
-Text GLabel 2850 2000 0    60   Input ~ 0
+Text GLabel 2650 2000 0    60   Input ~ 0
 D9
 NoConn ~ 3050 2100
@@
 $EndComp
 Text GLabel 2900 6300 0    60   Input ~ 0
-A4
+A2
 Text GLabel 1600 3600 0    60   Input ~ 0
 SCL
@@
 	4500 4400 4750 4400
 Wire Wire Line
-	2850 1900 3050 1900
-Wire Wire Line
-	2850 2000 3050 2000
-Wire Wire Line
 	3050 2500 3050 2700
 Wire Wire Line
@@
 	2250 2150 2250 2700
 Wire Wire Line
-	1600 4100 1900 4100
-Wire Wire Line
 	5250 1900 5250 2250
 Wire Wire Line
@@
 Wire Wire Line
 	8550 5050 8750 5050
+$Comp
+L R R10
+U 1 1 5A2EF399
+P 2850 1900
+F 0 "R10" V 2930 1900 50  0000 C CNN
+F 1 "1K" V 2850 1900 50  0000 C CNN
+F 2 "Resistors_ThroughHole:Resistor_Horizontal_RM7mm" V 2780 1900 50  0001 C CNN
+F 3 "" H 2850 1900 50  0000 C CNN
+	1    2850 1900
+	0    1    1    0
+$EndComp
+Wire Wire Line
+	3000 1900 3050 1900
+Wire Wire Line
+	2650 1900 2700 1900
+Wire Wire Line
+	2650 2000 3050 2000
+Text GLabel 1600 4300 0    60   Input ~ 0
+A2
+Wire Wire Line
+	1600 4300 1900 4300
 $EndSCHEMATC
