File: kicad/_saved_battlepoint.sch (KiCad schematic (older format))
At the start: 32 parts, among them J1 AUDIO, J2 RED_SWITCH, J3 BLU_SWITCH, J4 LED1, J5 LED2, J6 PWR_OPTION, J7 LED3, J8 LED4, P13 BTNS_IN, P14 OLED_OUT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

Commit message: routed
Parts:
- P17: footprint Pin_Headers:Pin_Header_Straight_1x04 -> Connectors_JST:JST_XH_B04B-XH-A_04x2.50mm_Straight
Changed lines of the file:
@@
 F 0 "P17" H 8100 3950 50  0000 C CNN
 F 1 "BTNS_OUT" V 8200 3700 50  0000 C CNN
-F 2 "Pin_Headers:Pin_Header_Straight_1x04" H 8100 3700 50  0001 C CNN
+F 2 "Connectors_JST:JST_XH_B04B-XH-A_04x2.50mm_Straight" H 8100 3700 50  0001 C CNN
 F 3 "" H 8100 3700 50  0000 C CNN
 	1    8100 3700
