File: tag_reader/kicad/esp32-board/esp32-board.kicad_sch (KiCad schematic)
At the start: 9 parts, among them J1 Conn_01x08_Pin, J2 Conn_01x04_Pin, J3 Conn_01x06_Pin, J4 Conn_01x15_Socket, J5 Conn_01x15_Socket, J6 Conn_01x15_Pin, J7 Conn_01x15_Pin, J8 Conn_01x06_Pin

Commit message: making board
Parts:
- removed J1: Conn_01x08_Pin, Connector_PinHeader_2.54mm:PinHeader_1x08_P2.54mm_Vertical, symbol Connector:Conn_01x08_Pin
- removed J2: Conn_01x04_Pin, Connector_PinHeader_2.54mm:PinHeader_1x04_P2.54mm_Horizontal, symbol Connector:Conn_01x04_Pin
- added J1, J9: Conn_01x03_Pin, Connector_PinHeader_2.54mm:PinHeader_1x03_P2.54mm_Horizontal, symbol Connector:Conn_01x03_Pin
Connections:
- net GND: now also J1.2 (Pin_2), J9.2 (Pin_2)
- net D27: now reaches J5.6 (Pin_6), J7.10 (Pin_10), U1.25 (D27)
- net D27: now also J1.1 (Pin_1), J9.3 (Pin_3)
- net D26: now reaches J5.7 (Pin_7), J7.9 (Pin_9), U1.24 (D26)
- net D26: now also J1.3 (Pin_3), J9.1 (Pin_1)

Commit message: compiling refactored, but not tested
Parts:
- removed J1, J9: Conn_01x03_Pin, Connector_PinHeader_2.54mm:PinHeader_1x03_P2.54mm_Horizontal, symbol Connector:Conn_01x03_Pin
- removed J3, J8: Conn_01x06_Pin, Connector_PinHeader_2.54mm:PinHeader_1x06_P2.54mm_Vertical, symbol Connector:Conn_01x06_Pin
- removed J4, J5: Conn_01x15_Socket, Connector_PinHeader_2.54mm:PinHeader_1x15_P2.54mm_Vertical, symbol Connector:Conn_01x15_Socket
- added J1: OLED, Connector_PinHeader_2.54mm:PinHeader_1x04_P2.54mm_Vertical, symbol Connector:Conn_01x04_Pin
- added J10: SW_LEFT, Connector_PinHeader_2.54mm:PinHeader_1x04_P2.54mm_Horizontal, symbol Connector:Conn_01x04_Pin
- added J12: LID, Connector_PinHeader_2.54mm:PinHeader_1x06_P2.54mm_Vertical, symbol Connector:Conn_01x06_Pin
- added J2: SW_RIGHT, Connector_PinHeader_2.54mm:PinHeader_1x04_P2.54mm_Horizontal, symbol Connector:Conn_01x04_Pin
- added J3: PWR, Connector_PinHeader_2.54mm:PinHeader_1x02_P2.54mm_Vertical, symbol Connector:Conn_01x02_Pin
- added J9: SPK, Connector_PinHeader_2.54mm:PinHeader_1x02_P2.54mm_Vertical, symbol Connector:Conn_01x02_Pin
Connections:
- net D26: now also J10.1 (Pin_1), J2.1 (Pin_1)
- net D27: now also J10.4 (Pin_4), J2.4 (Pin_4)
- net GND: now also J1.1 (Pin_1), J10.2 (Pin_2), J10.3 (Pin_3), J12.6 (Pin_6), J2.2 (Pin_2), J2.3 (Pin_3), J3.2 (Pin_2), J9.2 (Pin_2)
- net VCC: now also J1.2 (Pin_2), J12.5 (Pin_5), J3.1 (Pin_1)
- net SCL: now reaches J6.11 (Pin_11), U1.11 (D21/SCL)
- net SCL: now also J1.3 (Pin_3)
- net SDA: now reaches J6.14 (Pin_14), U1.14 (D22)
- net SDA: now also J1.4 (Pin_4)
- net RX2: now reaches J6.6 (Pin_6), U1.6 (RX2)
- net RX2: now also J12.2 (Pin_2)
- net TX2: now reaches J6.7 (Pin_7), U1.7 (TX2)
- net TX2: now also J12.1 (Pin_1)
- net LED1: now reaches J7.11 (Pin_11), U1.26 (D14)
- net LED1: now also J12.3 (Pin_3)
- net LED2: now reaches J7.12 (Pin_12), U1.27 (D12)
- net LED2: now also J12.4 (Pin_4)
- net SPK: now reaches J7.8 (Pin_8), U1.23 (D25)
- net SPK: now also J9.1 (Pin_1)
