File: payload/kicad/payload.kicad_pcb (KiCad board)
At the start: 2 copper layers, 81.3 x 81.3 mm, 12 parts, among them J1 MTR_CTRL, J10 SENS_LEFT, J11 SENS_RIGHT, J2 BTN_F2, J3 BTN_F3, J4 BTN_BCK, J5 BTN_F1, J6 Encoder, J7 OLED, J8 PWR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

Commit message: revive the payload. fiddling with mag sensors again
Other:
- net class Default removed
- net class Power removed
